Commit message: lidar_description : add urdf generation using python script

File: romea_lidar_description/urdf/lidar.xacro (robot description, xacro)
@@ -1,16 +1,6 @@
 <?xml version="1.0"?>
 <robot name="lidar" xmlns:xacro="http://www.ros.org/wiki/xacro" >
-<xacro:macro name="lidar_sensor" params="xyz rpy parent_link rate type model name">
-    <xacro:if value="${type == 'sick'}">
-       <xacro:if value="${'lms1' in model}">
-           <xacro:property name="specifications_file" value="$(find romea_lidar_description)/config/sick_lms1xx_${rate}hz_specifications.yaml" />
-           <xacro:property name="geometry_file" value="$(find romea_lidar_description)/config/sick_lms1xx_geometry.yaml" />
-       </xacro:if>
-       <xacro:if value="${'tim5' in model}">
-           <xacro:property name="specifications_file" value="$(find romea_lidar_description)/config/sick_tim5xx_specifications.yaml" />
-           <xacro:property name="geometry_file" value="$(find romea_lidar_description)/config/sick_tim5xx_geometry.yaml" />
-       </xacro:if>
-    </xacro:if>
-    <xacro:property name="specifications" value="${load_yaml(specifications_file)}"/>
+<xacro:macro name="lidar_sensor" params="prefix name type model parent_link xyz rpy mesh_visual rate minimal_azimut_angle maximal_azimut_angle minimal_range maximal_range samples">
+    <xacro:property name="geometry_file" value="$(find romea_lidar_description)/config/${type}_${model}_geometry.yaml" />
     <xacro:property name="geometry" value="${load_yaml(geometry_file)}"/>
     <xacro:property name="link_name" value="${prefix}${name}_link"/>
@@ -18,9 +8,4 @@
     <xacro:property name="controller_name" value="${prefix}${name}_controller"/>
     <xacro:property name="parent_link_name" value="${prefix}${parent_link}"/>
-    <xacro:property name="samples" value="${specifications['samples']}"/>
-    <xacro:property name="minimal_azimut_angle" value="${specifications['minimal_azimut_angle']/180.*pi}"/>
-    <xacro:property name="maximal_azimut_angle" value="${specifications['maximal_azimut_angle']/180.*pi}"/>
-    <xacro:property name="minimal_range" value="${specifications['minimal_range']}"/>
-    <xacro:property name="maximal_range" value="${specifications['maximal_range']}"/>
     <xacro:property name="mass" value="${geometry['mass']}"/>
     <xacro:property name="aabb_length" value="${geometry['aabb']['length']}"/>
@@ -30,4 +15,5 @@
     <xacro:property name="mesh_xyz" value="${geometry['mesh']['xyz']}"/>
     <xacro:property name="mesh_rpy" value="${geometry['mesh']['rpy']}"/>
+    <xacro:property name="mesh_scale" value="${geometry['mesh']['scale']}"/>
     <xacro:property name="mesh_filename" value="${geometry['mesh']['filename']}"/>
     <link name="${link_name}">
@@ -40,8 +26,16 @@
       </inertial>
       <visual>
-        <origin xyz="${mesh_xyz[0]} ${mesh_xyz[1]} ${mesh_xyz[2]}" rpy="${mesh_rpy[0]} ${mesh_rpy[1]} ${mesh_rpy[2]}" />
-          <geometry>
-            <mesh filename="${mesh_filename}" />
-          </geometry>
+        <xacro:if value="${mesh_visual == True}">
+           <origin xyz="${mesh_xyz[0]} ${mesh_xyz[1]} ${mesh_xyz[2]}" rpy="${mesh_rpy[0]} ${mesh_rpy[1]} ${mesh_rpy[2]}" />
+           <geometry>
+             <mesh filename="${mesh_filename}" scale="${mesh_scale[0]} ${mesh_scale[1]} ${mesh_scale[2]}" />
+           </geometry>
+        </xacro:if>
+        <xacro:if value="${mesh_visual == False}">
+           <origin xyz="${aabb_center[0]} ${aabb_center[1]} ${aabb_center[2]}" rpy="0 0 0" />
+           <geometry>
+             <box size="${aabb_length} ${aabb_width} ${aabb_height}" />
+           </geometry>
+        </xacro:if>
       </visual>
     <collision>
@@ -77,7 +71,10 @@
           </noise>
         </ray>
-        <plugin name="gazebo_ros_laser" filename="libgazebo_ros_laser.so">
-          <topicName>/${prefix}${name}/scan</topicName>
-          <frameName>${link_name}</frameName>
+        <plugin name="${name}" filename="libgazebo_ros_ray_sensor.so">
+          <ros>
+            <namespace>${prefix}${name}</namespace>
+            <remapping>~/out:=${name}/scan</remapping>
+          </ros>
+          <output_type>sensor_msgs/LaserScan</output_type>
         </plugin>
       </sensor>

File: romea_lidar_description/urdf/lidar3d.xacro (robot description, xacro)
@@ -1,5 +1,5 @@
 <?xml version="1.0"?>
 <robot name="lidar" xmlns:xacro="http://www.ros.org/wiki/xacro" >
-<xacro:macro name="lidar3d_sensor" params="xyz rpy parent_link rate type model name organize_cloud:=false gpu:=false">
+<xacro:macro name="lidar3d_sensor" params="xyz rpy parent_link rate type model name organize_cloud:=false gpu:=false prefix">
     <xacro:if value="${model == 'mrs1000'}">
         <xacro:property name="specifications_file" value="$(find romea_lidar_description)/config/sick_mrs1000_specifications.yaml" />

Commit message: description : mesh visual is avaible only if mes description is given in geometry file

File: romea_lidar_description/urdf/lidar.xacro (robot description, xacro)
@@ -2,29 +2,31 @@
 <robot name="lidar" xmlns:xacro="http://www.ros.org/wiki/xacro" >
 <xacro:macro name="lidar_sensor" params="prefix name type model parent_link xyz rpy mesh_visual rate minimal_azimut_angle maximal_azimut_angle minimal_range maximal_range samples">
-    <xacro:property name="geometry_file" value="$(find romea_lidar_description)/config/${type}_${model}_geometry.yaml" />
-    <xacro:property name="geometry" value="${load_yaml(geometry_file)}"/>
-    <xacro:property name="link_name" value="${prefix}${name}_link"/>
-    <xacro:property name="joint_name" value="${prefix}${name}_joint"/>
-    <xacro:property name="controller_name" value="${prefix}${name}_controller"/>
-    <xacro:property name="parent_link_name" value="${prefix}${parent_link}"/>
-    <xacro:property name="mass" value="${geometry['mass']}"/>
-    <xacro:property name="aabb_length" value="${geometry['aabb']['length']}"/>
-    <xacro:property name="aabb_width" value="${geometry['aabb']['width']}"/>
-    <xacro:property name="aabb_height" value="${geometry['aabb']['height']}"/>
-    <xacro:property name="aabb_center" value="${geometry['aabb']['center']}"/>
+  <xacro:property name="geometry_file" value="$(find romea_lidar_description)/config/${type}_${model}_geometry.yaml" />
+  <xacro:property name="geometry" value="${load_yaml(geometry_file)}"/>
+  <xacro:property name="link_name" value="${prefix}${name}_link"/>
+  <xacro:property name="joint_name" value="${prefix}${name}_joint"/>
+  <xacro:property name="controller_name" value="${prefix}${name}_controller"/>
+  <xacro:property name="parent_link_name" value="${prefix}${parent_link}"/>
+  <xacro:property name="mass" value="${geometry['mass']}"/>
+  <xacro:property name="aabb_length" value="${geometry['aabb']['length']}"/>
+  <xacro:property name="aabb_width" value="${geometry['aabb']['width']}"/>
+  <xacro:property name="aabb_height" value="${geometry['aabb']['height']}"/>
+  <xacro:property name="aabb_center" value="${geometry['aabb']['center']}"/>
+  <xacro:if value="${mesh_visual == True and 'mesh' in geometry}">
     <xacro:property name="mesh_xyz" value="${geometry['mesh']['xyz']}"/>
     <xacro:property name="mesh_rpy" value="${geometry['mesh']['rpy']}"/>
     <xacro:property name="mesh_scale" value="${geometry['mesh']['scale']}"/>
     <xacro:property name="mesh_filename" value="${geometry['mesh']['filename']}"/>
-    <link name="${link_name}">
-      <inertial>
-        <mass value="${mass}" />
-        <origin xyz="${aabb_center[0]} ${aabb_center[1]} ${aabb_center[2]}" />
-        <inertia ixx="${0.0833333 * mass * (aabb_width*aabb_width + aabb_height*aabb_height)}" ixy="0.0" ixz="0.0"
-          iyy="${0.0833333 * mass * (aabb_height*aabb_height + aabb_length*aabb_length)}" iyz="0.0"
-          izz="${0.0833333 * mass * (aabb_length*aabb_length + aabb_width*aabb_width)}" />
+  </xacro:if>
+  <link name="${link_name}">
+    <inertial>
+      <mass value="${mass}" />
+      <origin xyz="${aabb_center[0]} ${aabb_center[1]} ${aabb_center[2]}" />
+      <inertia ixx="${0.0833333 * mass * (aabb_width*aabb_width + aabb_height*aabb_height)}" ixy="0.0" ixz="0.0"
+               iyy="${0.0833333 * mass * (aabb_height*aabb_height + aabb_length*aabb_length)}" iyz="0.0"
+               izz="${0.0833333 * mass * (aabb_length*aabb_length + aabb_width*aabb_width)}" />
       </inertial>
       <visual>
-        <xacro:if value="${mesh_visual == True}">
+        <xacro:if value="${mesh_visual == True and 'mesh' in geometry}">
            <origin xyz="${mesh_xyz[0]} ${mesh_xyz[1]} ${mesh_xyz[2]}" rpy="${mesh_rpy[0]} ${mesh_rpy[1]} ${mesh_rpy[2]}" />
            <geometry>
@@ -32,5 +34,5 @@
            </geometry>
         </xacro:if>
-        <xacro:if value="${mesh_visual == False}">
+        <xacro:if value="${mesh_visual == False or 'mesh' not in geometry}">
            <origin xyz="${aabb_center[0]} ${aabb_center[1]} ${aabb_center[2]}" rpy="0 0 0" />
            <geometry>
@@ -80,10 +82,10 @@
       </sensor>
     </gazebo>
-    <joint name="${joint_name}" type="fixed">
-        <axis xyz="0 0 1" />
-        <origin xyz="${xyz}" rpy="${rpy}"/>
-        <parent link="${parent_link_name}"/>
-        <child link="${link_name}"/>
-    </joint>
+  <joint name="${joint_name}" type="fixed">
+    <axis xyz="0 0 1" />
+    <origin xyz="${xyz}" rpy="${rpy}"/>
+    <parent link="${parent_link_name}"/>
+    <child link="${link_name}"/>
+  </joint>
 </xacro:macro>
 </robot>

Commit message: update to take into account additional ros namespace in description

File: romea_lidar_description/urdf/lidar.xacro (robot description, xacro)
@@ -1,50 +1,55 @@
 <?xml version="1.0"?>
-<robot name="lidar" xmlns:xacro="http://www.ros.org/wiki/xacro" >
-<xacro:macro name="lidar_sensor" params="prefix name type model parent_link xyz rpy mesh_visual rate minimal_azimut_angle maximal_azimut_angle minimal_range maximal_range samples">
-  <xacro:property name="geometry_file" value="$(find romea_lidar_description)/config/${type}_${model}_geometry.yaml" />
-  <xacro:property name="geometry" value="${load_yaml(geometry_file)}"/>
-  <xacro:property name="link_name" value="${prefix}${name}_link"/>
-  <xacro:property name="joint_name" value="${prefix}${name}_joint"/>
-  <xacro:property name="controller_name" value="${prefix}${name}_controller"/>
-  <xacro:property name="parent_link_name" value="${prefix}${parent_link}"/>
-  <xacro:property name="mass" value="${geometry['mass']}"/>
-  <xacro:property name="aabb_length" value="${geometry['aabb']['length']}"/>
-  <xacro:property name="aabb_width" value="${geometry['aabb']['width']}"/>
-  <xacro:property name="aabb_height" value="${geometry['aabb']['height']}"/>
-  <xacro:property name="aabb_center" value="${geometry['aabb']['center']}"/>
-  <xacro:if value="${mesh_visual == True and 'mesh' in geometry}">
-    <xacro:property name="mesh_xyz" value="${geometry['mesh']['xyz']}"/>
-    <xacro:property name="mesh_rpy" value="${geometry['mesh']['rpy']}"/>
-    <xacro:property name="mesh_scale" value="${geometry['mesh']['scale']}"/>
-    <xacro:property name="mesh_filename" value="${geometry['mesh']['filename']}"/>
-  </xacro:if>
-  <link name="${link_name}">
-    <inertial>
-      <mass value="${mass}" />
-      <origin xyz="${aabb_center[0]} ${aabb_center[1]} ${aabb_center[2]}" />
-      <inertia ixx="${0.0833333 * mass * (aabb_width*aabb_width + aabb_height*aabb_height)}" ixy="0.0" ixz="0.0"
-               iyy="${0.0833333 * mass * (aabb_height*aabb_height + aabb_length*aabb_length)}" iyz="0.0"
-               izz="${0.0833333 * mass * (aabb_length*aabb_length + aabb_width*aabb_width)}" />
+<robot name="lidar" xmlns:xacro="http://www.ros.org/wiki/xacro">
+  <xacro:macro name="lidar_sensor"
+    params="prefix name type model parent_link xyz rpy mesh_visual rate minimal_azimut_angle maximal_azimut_angle minimal_range maximal_range samples ros_namespace">
+    <xacro:property name="geometry_file"
+      value="$(find romea_lidar_description)/config/${type}_${model}_geometry.yaml" />
+    <xacro:property name="geometry" value="${load_yaml(geometry_file)}" />
+    <xacro:property name="link_name" value="${prefix}${name}_link" />
+    <xacro:property name="joint_name" value="${prefix}${name}_joint" />
+    <xacro:property name="controller_name" value="${prefix}${name}_controller" />
+    <xacro:property name="parent_link_name" value="${prefix}${parent_link}" />
+    <xacro:property name="mass" value="${geometry['mass']}" />
+    <xacro:property name="aabb_length" value="${geometry['aabb']['length']}" />
+    <xacro:property name="aabb_width" value="${geometry['aabb']['width']}" />
+    <xacro:property name="aabb_height" value="${geometry['aabb']['height']}" />
+    <xacro:property name="aabb_center" value="${geometry['aabb']['center']}" />
+    <xacro:if value="${mesh_visual == True and 'mesh' in geometry}">
+      <xacro:property name="mesh_xyz" value="${geometry['mesh']['xyz']}" />
+      <xacro:property name="mesh_rpy" value="${geometry['mesh']['rpy']}" />
+      <xacro:property name="mesh_scale" value="${geometry['mesh']['scale']}" />
+      <xacro:property name="mesh_filename" value="${geometry['mesh']['filename']}" />
+    </xacro:if>
+    <link name="${link_name}">
+      <inertial>
+        <mass value="${mass}" />
+        <origin xyz="${aabb_center[0]} ${aabb_center[1]} ${aabb_center[2]}" />
+        <inertia ixx="${0.0833333 * mass * (aabb_width*aabb_width + aabb_height*aabb_height)}"
+          ixy="0.0" ixz="0.0"
+          iyy="${0.0833333 * mass * (aabb_height*aabb_height + aabb_length*aabb_length)}" iyz="0.0"
+          izz="${0.0833333 * mass * (aabb_length*aabb_length + aabb_width*aabb_width)}" />
       </inertial>
       <visual>
         <xacro:if value="${mesh_visual == True and 'mesh' in geometry}">
-           <origin xyz="${mesh_xyz[0]} ${mesh_xyz[1]} ${mesh_xyz[2]}" rpy="${mesh_rpy[0]} ${mesh_rpy[1]} ${mesh_rpy[2]}" />
-           <geometry>
-             <mesh filename="${mesh_filename}" scale="${mesh_scale[0]} ${mesh_scale[1]} ${mesh_scale[2]}" />
-           </geometry>
+          <origin xyz="${mesh_xyz[0]} ${mesh_xyz[1]} ${mesh_xyz[2]}"
+            rpy="${mesh_rpy[0]} ${mesh_rpy[1]} ${mesh_rpy[2]}" />
+          <geometry>
+            <mesh filename="${mesh_filename}"
+              scale="${mesh_scale[0]} ${mesh_scale[1]} ${mesh_scale[2]}" />
+          </geometry>
         </xacro:if>
         <xacro:if value="${mesh_visual == False or 'mesh' not in geometry}">
-           <origin xyz="${aabb_center[0]} ${aabb_center[1]} ${aabb_center[2]}" rpy="0 0 0" />
-           <geometry>
-             <box size="${aabb_length} ${aabb_width} ${aabb_height}" />
-           </geometry>
+          <origin xyz="${aabb_center[0]} ${aabb_center[1]} ${aabb_center[2]}" rpy="0 0 0" />
+          <geometry>
+            <box size="${aabb_length} ${aabb_width} ${aabb_height}" />
+          </geometry>
         </xacro:if>
       </visual>
-    <collision>
-      <origin xyz="${aabb_center[0]} ${aabb_center[1]} ${aabb_center[2]}" rpy="0 0 0" />
-      <geometry>
-        <box size="${aabb_length} ${aabb_width} ${aabb_height}" />
-      </geometry>
-    </collision>
+      <collision>
+        <origin xyz="${aabb_center[0]} ${aabb_center[1]} ${aabb_center[2]}" rpy="0 0 0" />
+        <geometry>
+          <box size="${aabb_length} ${aabb_width} ${aabb_height}" />
+        </geometry>
+      </collision>
     </link>
     <gazebo reference="${link_name}">
@@ -73,8 +78,8 @@
           </noise>
         </ray>
-        <plugin name="${name}" filename="libgazebo_ros_ray_sensor.so">
+        <plugin name="driver" filename="libgazebo_ros_ray_sensor.so">
           <ros>
-            <!-- <namespace>${prefix}${name}</namespace> --> <!-- not working -->
-            <remapping>~/out:=${name}/scan</remapping>
+            <namespace>${ros_namespace}</namespace>
+            <remapping>~/out:=scan</remapping>
           </ros>
           <output_type>sensor_msgs/LaserScan</output_type>
@@ -82,10 +87,10 @@
       </sensor>
     </gazebo>
-  <joint name="${joint_name}" type="fixed">
-    <axis xyz="0 0 1" />
-    <origin xyz="${xyz}" rpy="${rpy}"/>
-    <parent link="${parent_link_name}"/>
-    <child link="${link_name}"/>
-  </joint>
-</xacro:macro>
+    <joint name="${joint_name}" type="fixed">
+      <axis xyz="0 0 1" />
+      <origin xyz="${xyz}" rpy="${rpy}" />
+      <parent link="${parent_link_name}" />
+      <child link="${link_name}" />
+    </joint>
+  </xacro:macro>
 </robot>
