Commit message: description: set Blue color to bounding box
Signed-off-by: Jean Laneurit <jean.laneurit@inrae.fr>

File: romea_lidar_description/urdf/lidar2D.xacro (robot description, xacro)
@@ -67,4 +67,5 @@
     </link>
     <gazebo reference="${link_name}">
+      <material>Gazebo/Blue</material>
       <sensor type="ray" name="${prefix}${name}">
         <pose>0 0 0 0 0 0</pose>

File: romea_lidar_description/urdf/lidar3D.xacro (robot description, xacro)
@@ -72,4 +72,5 @@
     <gazebo reference="${link_name}">
       <!-- <xacro:if value="${gpu}"> -->
+      <material>Gazebo/Blue</material>
       <sensor type="gpu_ray" name="${prefix}${name}">
         <pose>0 0 0 0 0 0</pose>

Commit message: description: add lidar simulation xacro files
Signed-off-by: Jean Laneurit <jean.laneurit@inrae.fr>

File: romea_lidar_description/urdf/lidar2D.xacro (robot description, xacro)
@@ -11,26 +11,23 @@
     <xacro:property name="parent_link_name"
       value="${prefix}${parent_link}" />
-    <xacro:property name="minimal_azimut_angle"
-      value="${configuration['minimal_azimut_angle']/180.*pi}" />
-    <xacro:property name="maximal_azimut_angle"
-      value="${configuration['maximal_azimut_angle']/180.*pi}" />
-    <xacro:property name="minimal_range"
-      value="${configuration['minimal_range']}" />
-    <xacro:property name="maximal_range"
-      value="${configuration['maximal_range']}" />
-    <xacro:property name="samples"
-      value="${configuration['samples']}" />
-    <xacro:property name="rate"
-      value="${configuration['rate']}" />
-    <xacro:property name="mass" value="${geometry['mass']}" />
-    <xacro:property name="aabb_length" value="${geometry['aabb']['length']}" />
-    <xacro:property name="aabb_width" value="${geometry['aabb']['width']}" />
-    <xacro:property name="aabb_height" value="${geometry['aabb']['height']}" />
-    <xacro:property name="aabb_center" value="${geometry['aabb']['center']}" />
+    <xacro:property name="mass"
+      value="${geometry['mass']}" />
+    <xacro:property name="aabb_length"
+      value="${geometry['aabb']['length']}" />
+    <xacro:property name="aabb_width"
+      value="${geometry['aabb']['width']}" />
+    <xacro:property name="aabb_height"
+      value="${geometry['aabb']['height']}" />
+    <xacro:property name="aabb_center"
+      value="${geometry['aabb']['center']}" />
     <xacro:if value="${mesh_visual == True and 'mesh' in geometry}">
-      <xacro:property name="mesh_xyz" value="${geometry['mesh']['xyz']}" />
-      <xacro:property name="mesh_rpy" value="${geometry['mesh']['rpy']}" />
-      <xacro:property name="mesh_scale" value="${geometry['mesh']['scale']}" />
-      <xacro:property name="mesh_filename" value="${geometry['mesh']['filename']}" />
+      <xacro:property name="mesh_xyz"
+        value="${geometry['mesh']['xyz']}" />
+      <xacro:property name="mesh_rpy"
+        value="${geometry['mesh']['rpy']}" />
+      <xacro:property name="mesh_scale"
+        value="${geometry['mesh']['scale']}" />
+      <xacro:property name="mesh_filename"
+        value="${geometry['mesh']['filename']}" />
     </xacro:if>
     <link name="${link_name}">
@@ -66,40 +63,14 @@
       </collision>
     </link>
-    <gazebo reference="${link_name}">
-      <material>Gazebo/Blue</material>
-      <sensor type="ray" name="${prefix}${name}">
-        <pose>0 0 0 0 0 0</pose>
-        <visualize>true</visualize>
-        <update_rate>${rate}</update_rate>
-        <ray>
-          <scan>
-            <horizontal>
-              <samples>${samples}</samples>
-              <resolution>1</resolution>
-              <min_angle>${minimal_azimut_angle}</min_angle>
-              <max_angle>${maximal_azimut_angle}</max_angle>
-            </horizontal>
-          </scan>
-          <range>
-            <min>${minimal_range}</min>
-            <max>${maximal_range}</max>
-            <resolution>0.01</resolution>
-          </range>
-          <noise>
-            <type>gaussian</type>
-            <mean>0.0</mean>
-            <stddev>0.001</stddev>
-          </noise>
-        </ray>
-        <plugin name="driver" filename="libgazebo_ros_ray_sensor.so">
-          <ros>
-            <namespace>${ros_namespace}</namespace>
-            <remapping>~/out:=scan</remapping>
-          </ros>
-          <frame_name>${link_name}</frame_name>
-          <output_type>sensor_msgs/LaserScan</output_type>
-        </plugin>
-      </sensor>
-    </gazebo>
+    <xacro:if value="${'simulation' in  mode}">
+      <xacro:include filename="$(find romea_lidar_description)/urdf/lidar2D.simulation.xacro" />
+      <xacro:lidar2d_sensor_simulation
+        prefix="${prefix}"
+        mode="${mode}"
+        name="${name}"
+        link_name="${link_name}"
+        configuration="${configuration}"
+        ros_namespace="${ros_namespace}"/>
+    </xacro:if>
     <joint name="${joint_name}" type="fixed">
       <axis xyz="0 0 1" />

File: romea_lidar_description/urdf/lidar3D.xacro (robot description, xacro)
@@ -3,38 +3,31 @@
   <xacro:macro name="lidar3d_sensor"
     params="prefix mode name configuration geometry xyz rpy parent_link mesh_visual ros_namespace ">
-    <xacro:property name="link_name" value="${prefix}${name}_link" />
-    <xacro:property name="joint_name" value="${prefix}${name}_joint" />
-    <xacro:property name="controller_name" value="${prefix}${name}_controller" />
-    <xacro:property name="parent_link_name" value="${prefix}${parent_link}" />
-    <xacro:property name="samples"
-      value="${configuration['samples']}" />
-    <xacro:property name="minimal_azimut_angle"
-      value="${configuration['minimal_azimut_angle']/180.*pi}" />
-    <xacro:property name="maximal_azimut_angle"
-      value="${configuration['maximal_azimut_angle']/180.*pi}" />
-    <xacro:property name="lasers"
-      value="${configuration['lasers']}" />
-    <xacro:property name="minimal_elevation_angle"
-      value="${configuration['minimal_elevation_angle']/180.*pi}" />
-    <xacro:property name="maximal_elevation_angle"
-      value="${configuration['maximal_elevation_angle']/180.*pi}" />
-    <xacro:property name="minimal_range"
-      value="${configuration['minimal_range']}" />
-    <xacro:property name="maximal_range"
-      value="${configuration['maximal_range']}" />
-    <xacro:property name="range_std"
-      value="${configuration['range_std']}" />
-    <xacro:property name="rate"
-      value="${configuration['rate']}" />
-    <xacro:property name="mass" value="${geometry['mass']}" />
-    <xacro:property name="aabb_length" value="${geometry['aabb']['length']}" />
-    <xacro:property name="aabb_width" value="${geometry['aabb']['width']}" />
-    <xacro:property name="aabb_height" value="${geometry['aabb']['height']}" />
-    <xacro:property name="aabb_center" value="${geometry['aabb']['center']}" />
+    <xacro:property name="link_name"
+      value="${prefix}${name}_link" />
+    <xacro:property name="joint_name"
+      value="${prefix}${name}_joint" />
+    <xacro:property name="controller_name"
+      value="${prefix}${name}_controller" />
+    <xacro:property name="parent_link_name"
+      value="${prefix}${parent_link}" />
+    <xacro:property name="mass"
+      value="${geometry['mass']}" />
+    <xacro:property name="aabb_length"
+      value="${geometry['aabb']['length']}" />
+    <xacro:property name="aabb_width"
+      value="${geometry['aabb']['width']}" />
+    <xacro:property name="aabb_height"
+      value="${geometry['aabb']['height']}" />
+    <xacro:property name="aabb_center"
+      value="${geometry['aabb']['center']}" />
     <xacro:if value="${mesh_visual == True and 'mesh' in geometry}">
-      <xacro:property name="mesh_xyz" value="${geometry['mesh']['xyz']}" />
-      <xacro:property name="mesh_rpy" value="${geometry['mesh']['rpy']}" />
-      <xacro:property name="mesh_scale" value="${geometry['mesh']['scale']}" />
-      <xacro:property name="mesh_filename" value="${geometry['mesh']['filename']}" />
+      <xacro:property name="mesh_xyz"
+        value="${geometry['mesh']['xyz']}" />
+      <xacro:property name="mesh_rpy"
+        value="${geometry['mesh']['rpy']}" />
+      <xacro:property name="mesh_scale"
+        value="${geometry['mesh']['scale']}" />
+      <xacro:property name="mesh_filename"
+        value="${geometry['mesh']['filename']}" />
     </xacro:if>
     <link name="${link_name}">
@@ -70,89 +63,14 @@
       </collision>
     </link>
-    <gazebo reference="${link_name}">
-      <!-- <xacro:if value="${gpu}"> -->
-      <material>Gazebo/Blue</material>
-      <sensor type="gpu_ray" name="${prefix}${name}">
-        <pose>0 0 0 0 0 0</pose>
-        <visualize>true</visualize>
-        <update_rate>${rate}</update_rate>
-        <ray>
-          <scan>
-            <horizontal>
-              <samples>${samples}</samples>
-              <resolution>1</resolution>
-              <min_angle>${minimal_azimut_angle}</min_angle>
-              <max_angle>${maximal_azimut_angle}</max_angle>
-            </horizontal>
-            <vertical>
-              <samples>${lasers}</samples>
-              <resolution>1</resolution>
-              <min_angle>${minimal_elevation_angle}</min_angle>
-              <max_angle>${maximal_elevation_angle}</max_angle>
-            </vertical>
-          </scan>
-          <range>
-            <min>${minimal_range}</min>
-            <max>${maximal_range}</max>
-            <resolution>0.001</resolution>
-          </range>
-          <noise>
-            <type>gaussian</type>
-            <mean>0.0</mean>
-            <stddev>${range_std}</stddev>
-          </noise>
-        </ray>
-        <plugin name="driver" filename="libgazebo_ros_ray_sensor.so">
-          <ros>
-            <namespace>${ros_namespace}</namespace>
-            <remapping>~/out:=points</remapping>
-          </ros>
-          <frame_name>${link_name}</frame_name>
-          <output_type>sensor_msgs/PointCloud2</output_type>
-        </plugin>
-      </sensor>
-      <!-- </xacro:if> -->
-      <!-- <xacro:unless value="${gpu}">
-        <sensor type="ray" name="${prefix}${name}">
-          <pose>0 0 0 0 0 0</pose>
-          <visualize>true</visualize>
-          <update_rate>${rate}</update_rate>
-          <ray>
-            <scan>
-              <horizontal>
-                <samples>${samples}</samples>
-                <resolution>1</resolution>
-                <min_angle>${minimal_azimut_angle}</min_angle>
-                <max_angle>${maximal_azimut_angle}</max_angle>
-              </horizontal>
-              <vertical>
-                <samples>${lasers}</samples>
-                <resolution>1</resolution>
-                <min_angle>${minimal_elevation_angle}</min_angle>
-                <max_angle>${maximal_elevation_angle}</max_angle>
-              </vertical>
-            </scan>
-            <range>
-              <min>${minimal_range}</min>
-              <max>${maximal_range}</max>
-              <resolution>0.001</resolution>
-            </range>
-            <noise>
-              <type>gaussian</type>
-              <mean>0.0</mean>
-              <stddev>${range_std}</stddev>
-            </noise>
-          </ray>
-          <plugin name="gazebo_ros_laser_controller" filename="libgazebo_ros_romea_lidar3d.so">
-            <topicName>/${prefix}${name}/points</topicName>
-            <frameName>${link_name}</frameName>
-            <organize_cloud>${organize_cloud}</organize_cloud>
-            <min_range>${minimal_range}</min_range>
-            <max_range>${maximal_range}</max_range>
-            <gaussianNoise>${range_std}</gaussianNoise>
-          </plugin>
-        </sensor>
-      </xacro:unless>-->
-    </gazebo>
+    <xacro:if value="${'simulation' in  mode}">
+      <xacro:include filename="$(find romea_lidar_description)/urdf/lidar3D.simulation.xacro" />
+      <xacro:lidar3d_sensor_simulation
+        prefix="${prefix}"
+        mode="${mode}"
+        name="${name}"
+        link_name="${link_name}"
+        configuration="${configuration}"
+        ros_namespace="${ros_namespace}"/>
+    </xacro:if>
     <joint name="${joint_name}" type="fixed">
       <axis xyz="0 0 1" />

Commit message: disable collision in URDF

File: romea_lidar_description/urdf/lidar2D.xacro (robot description, xacro)
@@ -56,10 +56,10 @@
         </xacro:if>
       </visual>
-      <collision>
+      <!-- <collision>
         <origin xyz="${aabb_center[0]} ${aabb_center[1]} ${aabb_center[2]}" rpy="0 0 0" />
         <geometry>
           <box size="${aabb_length} ${aabb_width} ${aabb_height}" />
         </geometry>
-      </collision>
+      </collision> -->
     </link>
     <xacro:if value="${'simulation' in  mode}">

File: romea_lidar_description/urdf/lidar3D.xacro (robot description, xacro)
@@ -56,10 +56,10 @@
         </xacro:if>
       </visual>
-      <collision>
+      <!-- <collision>
         <origin xyz="${aabb_center[0]} ${aabb_center[1]} ${aabb_center[2]}" rpy="0 0 0" />
         <geometry>
           <box size="${aabb_length} ${aabb_width} ${aabb_height}" />
         </geometry>
-      </collision>
+      </collision> -->
     </link>
     <xacro:if value="${'simulation' in  mode}">
