Commit message: remove parent_link xyz rpy parmeters in xacro macro and set them in the configuration file
Signed-off-by: jean.laneurit <jean.laneurit@inrae.fr>

File: romea_lidar_description/urdf/lidar2D.simulation.xacro (robot description, xacro)
@@ -4,7 +4,7 @@
     params="prefix mode link_name name configuration ros_namespace">
     <xacro:property name="minimal_azimut_angle"
-      value="${configuration['minimal_azimut_angle']}" />
+      value="${configuration['minimal_azimut_angle']/180.*pi}" />
     <xacro:property name="maximal_azimut_angle"
-      value="${configuration['maximal_azimut_angle']}" />
+      value="${configuration['maximal_azimut_angle']/180.*pi}" />
     <xacro:property name="minimal_range"
       value="${configuration['minimal_range']}" />

File: romea_lidar_description/urdf/lidar2D.xacro (robot description, xacro)
@@ -2,5 +2,5 @@
 <robot name="lidar" xmlns:xacro="http://www.ros.org/wiki/xacro">
   <xacro:macro name="lidar2d_sensor"
-    params="prefix mode name configuration geometry parent_link xyz rpy mesh_visual ros_namespace">
+    params="prefix mode name configuration geometry mesh_visual ros_namespace">
     <xacro:property name="link_name"
       value="${prefix}${name}_link" />
@@ -10,5 +10,9 @@
       value="${prefix}${name}_controller" />
     <xacro:property name="parent_link_name"
-      value="${prefix}${parent_link}" />
+      value="${prefix}${configuration['parent_link']}" />
+    <xacro:property name="xyz"
+      value="${configuration['xyz']}" />
+    <xacro:property name="rpy"
+      value="${configuration['rpy']}" />
     <xacro:property name="mass"
       value="${geometry['mass']}" />
@@ -43,5 +47,5 @@
         <xacro:if value="${mesh_visual == True and 'mesh' in geometry}">
           <origin xyz="${mesh_xyz[0]} ${mesh_xyz[1]} ${mesh_xyz[2]}"
-            rpy="${mesh_rpy[0]} ${mesh_rpy[1]} ${mesh_rpy[2]}" />
+            rpy="${mesh_rpy[0]/180.*pi} ${mesh_rpy[1]/180.*pi} ${mesh_rpy[2]/180.*pi}" />
           <geometry>
             <mesh filename="${mesh_filename}"
@@ -71,9 +75,10 @@
         link_name="${link_name}"
         configuration="${configuration}"
-        ros_namespace="${ros_namespace}"/>
+        ros_namespace="${ros_namespace}" />
     </xacro:if>
     <joint name="${joint_name}" type="fixed">
       <axis xyz="0 0 1" />
-      <origin xyz="${xyz}" rpy="${rpy}" />
+      <origin xyz="${xyz[0]} ${xyz[1]} ${xyz[2]}"
+        rpy="${rpy[0]/180.*pi} ${rpy[1]/180.*pi} ${rpy[2]/180.*pi}" />
       <parent link="${parent_link_name}" />
       <child link="${link_name}" />

File: romea_lidar_description/urdf/lidar3D.simulation.xacro (robot description, xacro)
@@ -6,13 +6,13 @@
       value="${configuration['samples']}" />
     <xacro:property name="minimal_azimut_angle"
-      value="${configuration['minimal_azimut_angle']}" />
+      value="${configuration['minimal_azimut_angle']/180.*pi}" />
     <xacro:property name="maximal_azimut_angle"
-      value="${configuration['maximal_azimut_angle']}" />
+      value="${configuration['maximal_azimut_angle']/180.*pi}" />
     <xacro:property name="lasers"
       value="${configuration['lasers']}" />
     <xacro:property name="minimal_elevation_angle"
-      value="${configuration['minimal_elevation_angle']}" />
+      value="${configuration['minimal_elevation_angle']/180.*pi}" />
     <xacro:property name="maximal_elevation_angle"
-      value="${configuration['maximal_elevation_angle']}" />
+      value="${configuration['maximal_elevation_angle']/180.*pi}" />
     <xacro:property name="minimal_range"
       value="${configuration['minimal_range']}" />

File: romea_lidar_description/urdf/lidar3D.xacro (robot description, xacro)
@@ -2,5 +2,5 @@
 <robot name="lidar" xmlns:xacro="http://www.ros.org/wiki/xacro">
   <xacro:macro name="lidar3d_sensor"
-    params="prefix mode name configuration geometry xyz rpy parent_link mesh_visual ros_namespace ">
+    params="prefix mode name configuration geometry mesh_visual ros_namespace ">
     <xacro:property name="link_name"
       value="${prefix}${name}_link" />
@@ -10,5 +10,9 @@
       value="${prefix}${name}_controller" />
     <xacro:property name="parent_link_name"
-      value="${prefix}${parent_link}" />
+      value="${prefix}${configuration['parent_link']}" />
+    <xacro:property name="xyz"
+      value="${configuration['xyz']}" />
+    <xacro:property name="rpy"
+      value="${configuration['rpy']}" />
     <xacro:property name="mass"
       value="${geometry['mass']}" />
@@ -43,5 +47,5 @@
         <xacro:if value="${mesh_visual == True and 'mesh' in geometry}">
           <origin xyz="${mesh_xyz[0]} ${mesh_xyz[1]} ${mesh_xyz[2]}"
-            rpy="${mesh_rpy[0]} ${mesh_rpy[1]} ${mesh_rpy[2]}" />
+            rpy="${mesh_rpy[0]/180.*pi} ${mesh_rpy[1]/180.*pi} ${mesh_rpy[2]/180.*pi}" />
           <geometry>
             <mesh filename="${mesh_filename}"
@@ -71,5 +75,5 @@
         link_name="${link_name}"
         configuration="${configuration}"
-        ros_namespace="${ros_namespace}"/>
+        ros_namespace="${ros_namespace}" />
     </xacro:if>
     <!-- <joint name="${joint_name}" type="fixed">
@@ -83,5 +87,6 @@
         effort="10000000" velocity="1000000" />
       <axis xyz="0 0 1" />
-      <origin xyz="${xyz}" rpy="${rpy}" />
+      <origin xyz="${xyz[0]} ${xyz[1]} ${xyz[2]}"
+        rpy="${rpy[0]/180.*pi} ${rpy[1]/180.*pi} ${rpy[2]/180.*pi}" />
       <parent link="${parent_link_name}" />
       <child link="${link_name}" />

Commit message: description: add option to create standalone urdf description
Signed-off-by: Jean Laneurit <jean.laneurit@inrae.fr>

File: romea_lidar_description/urdf/lidar2D.simulation.xacro (robot description, xacro)
@@ -18,5 +18,5 @@
       <gazebo reference="${link_name}">
         <material>Gazebo/Blue</material>
-        <sensor type="ray" name="${prefix}${name}">
+        <sensor type="gpu_ray" name="${prefix}${name}">
           <pose>0 0 0 0 0 0</pose>
           <visualize>true</visualize>

File: romea_lidar_description/urdf/lidar2D.xacro (robot description, xacro)
@@ -2,5 +2,5 @@
 <robot name="lidar" xmlns:xacro="http://www.ros.org/wiki/xacro">
   <xacro:macro name="lidar2d_sensor"
-    params="prefix mode name configuration geometry mesh_visual ros_namespace">
+    params="prefix mode name configuration geometry mesh_visual ros_namespace standalone">
     <xacro:property name="link_name"
       value="${prefix}${name}_link" />
@@ -52,4 +52,7 @@
               scale="${mesh_scale[0]} ${mesh_scale[1]} ${mesh_scale[2]}" />
           </geometry>
+          <material name="lidar_color">
+            <color rgba="0 0 1 1"/>
+          </material>
         </xacro:if>
         <xacro:if value="${mesh_visual == False or 'mesh' not in geometry}">
@@ -77,11 +80,13 @@
         ros_namespace="${ros_namespace}" />
     </xacro:if>
-    <joint name="${joint_name}" type="fixed">
-      <axis xyz="0 0 1" />
-      <origin xyz="${xyz[0]} ${xyz[1]} ${xyz[2]}"
-        rpy="${rpy[0]/180.*pi} ${rpy[1]/180.*pi} ${rpy[2]/180.*pi}" />
-      <parent link="${parent_link_name}" />
-      <child link="${link_name}" />
-    </joint>
+    <xacro:if value="${standalone == False}">
+      <joint name="${joint_name}" type="fixed">
+        <axis xyz="0 0 1" />
+        <origin xyz="${xyz[0]} ${xyz[1]} ${xyz[2]}"
+          rpy="${rpy[0]/180.*pi} ${rpy[1]/180.*pi} ${rpy[2]/180.*pi}" />
+        <parent link="${parent_link_name}" />
+        <child link="${link_name}" />
+      </joint>
+    </xacro:if>
   </xacro:macro>
 </robot>

File: romea_lidar_description/urdf/lidar3D.xacro (robot description, xacro)
@@ -2,5 +2,5 @@
 <robot name="lidar" xmlns:xacro="http://www.ros.org/wiki/xacro">
   <xacro:macro name="lidar3d_sensor"
-    params="prefix mode name configuration geometry mesh_visual ros_namespace ">
+    params="prefix mode name configuration geometry mesh_visual ros_namespace standalone">
     <xacro:property name="link_name"
       value="${prefix}${name}_link" />
@@ -77,11 +77,13 @@
         ros_namespace="${ros_namespace}" />
     </xacro:if>
-    <joint name="${joint_name}" type="fixed">
-      <axis xyz="0 0 1" />
-      <origin xyz="${xyz[0]} ${xyz[1]} ${xyz[2]}"
-        rpy="${rpy[0]/180.*pi} ${rpy[1]/180.*pi} ${rpy[2]/180.*pi}" />
-      <parent link="${parent_link_name}" />
-      <child link="${link_name}" />
-    </joint>
+    <xacro:if value="${standalone == False}">
+      <joint name="${joint_name}" type="fixed">
+        <axis xyz="0 0 1" />
+        <origin xyz="${xyz[0]} ${xyz[1]} ${xyz[2]}"
+          rpy="${rpy[0]/180.*pi} ${rpy[1]/180.*pi} ${rpy[2]/180.*pi}" />
+        <parent link="${parent_link_name}" />
+        <child link="${link_name}" />
+      </joint>
+    </xacro:if>
   </xacro:macro>
 </robot>
